File: hardware/drv8701-dual-12v/KiCad_Import_5/DRV8701_DUAL_12V.sch (KiCad schematic (older format))
At the start: 38 parts, among them CN1 XT30UPB-M, CN2 XT30UPB-M, CN3 XH2.54-4P, P2 XT30UPB-M, Q1 TPH1R403NL, Q2 TPH1R403NL, Q3 TPH1R403NL, Q4 TPH1R403NL, Q5 TPH1R403NL, Q6 TPH1R403NL, Q7 TPH1R403NL, Q8 TPH1R403NL, U1 DRV8701ERGET, U2 DRV8701ERGET, U5 SS12D10G4

Commit message: Rework DRV8701 Rev B power control and manual PCB layout
Parts:
- added C18: 4.7uF, DRV8701_Custom:C_0805_2012Metric, symbol DRV8701_Custom:C
- added C19: 10nF, DRV8701_Custom:C_0603_1608Metric, symbol DRV8701_Custom:C
- added R10: 100kΩ, DRV8701_Custom:R_0603_1608Metric, symbol DRV8701_Custom:R
- added R11: 33kΩ, DRV8701_Custom:R_0603_1608Metric, symbol DRV8701_Custom:R
- added R12: 40.2kΩ, DRV8701_Custom:R_0603_1608Metric, symbol DRV8701_Custom:R
- added SW1: SS12D10G4, DRV8701_Custom:SS12D10G4, symbol DRV8701_Custom:SS12D10G4
- added U6: TPS25910RSAR, DRV8701_Custom:TPS25910_RSA16, symbol DRV8701_Custom:TPS25910RSAR
- P2: Source Original PDF; connections and values retained -> Original PDF; Rev B authorized P2.1 input rail split
Connections:
- net GND: now also C18.2, C19.2, R11.2, R12.2, SW1.3 (ON), U6.13 (GND), U6.14 (GND), U6.17 (EP), U6.5 (GND), U6.6 (GND), U6.8 (GND), U6.9 (GND)
- net VM: now also U6.10 (OUT), U6.11 (OUT), U6.12 (OUT); no longer P2.1 (+12V_RAW)
- new net PWR_EN: R10.2, R11.1, SW1.2 (COM), U6.16 (EN)
- new net PWR_GATE: C19.1, U6.4 (GATE)
- new net PWR_ILIM: R12.1, U6.7 (ILIM)
- new net VM_RAW: C18.1, P2.1 (+12V_RAW), R10.1, U6.1 (IN), U6.2 (IN), U6.3 (IN)
- no-connect marks 7 -> 9
Other:
- note added: "5A nominal limit; about 11ms typical start"
- note added: "OFF chip input standby: 2.5mA typ / 4mA max"
- note added: "REV B MAIN HIGH-SIDE POWER"
- note added: "REV B: authorized main power addition; all original values retained; only P2.1 changed to VM_RAW."
- note added: "SW1 ON = EN low; OFF = divider high"
- note added: "VREF/IDRIVE tied to AVDD; SP/SN grounded; nFAULT/SNSOUT/SO NC. U6 adds a shared supply current limit."
- note removed: "SOURCE-FAITHFUL DESIGN — values and connections intentionally retained; no hardware validation."
- note removed: "VREF/IDRIVE tied to AVDD; SP/SN grounded; nFAULT/SNSOUT/SO NC. No external current sensing or limit."
- moved on the sheet: CN1, CN2
